File: layout/binaryclock.brd (EAGLE design)
At the start: 100 x 50 mm, 84 parts, among them IC1 LP2985, IC3 STM32F10XCXT6, Q1 BSS84, Q4 BC807-16SMD, X1 MINI-USB-SHIELD-UX60-MB-5ST

Commit message: split layout into three frames
Connections:
- removed net N$6: C3.1, IC3.4, XTAL.4
- removed net N$7: C2.2, IC3.3, XTAL.1
- new net OSC1: C2.2, XTAL.1
- new net OSC2: C3.1, XTAL.4
Routing:
- net OSC2: track 0.00 -> 2.27 mm
- net N$6: track 2.27 -> 0.00 mm
- net OSC1: track 0.00 -> 2.27 mm
- net N$7: track 2.27 -> 0.00 mm
Changed lines of the file:
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@@
 <contactref element="IC3" pad="1"/>
 </signal>
-<signal name="N$6">
-<contactref element="IC3" pad="4"/>
+<signal name="OSC2">
 <contactref element="C3" pad="1"/>
 <contactref element="XTAL" pad="4"/>
 <wire x1="68.91" y1="37.89" x2="71.12" y2="37.89" width="0.4064" layer="16"/>
 <wire x1="71.12" y1="37.89" x2="71.12" y2="37.83" width="0.4064" layer="16"/>
-<wire x1="68.91" y1="37.89" x2="67.67" y2="53.65" width="0" layer="19" extent="16-16"/>
 </signal>
-<signal name="N$7">
+<signal name="OSC1">
 <contactref element="C2" pad="2"/>
-<contactref element="IC3" pad="3"/>
 <contactref element="XTAL" pad="1"/>
 <wire x1="65.71" y1="37.89" x2="63.5" y2="37.89" width="0.4064" layer="16"/>
 <wire x1="63.5" y1="37.89" x2="63.5" y2="37.83" width="0.4064" layer="16"/>
-<wire x1="65.71" y1="37.89" x2="68.17" y2="53.65" width="0" layer="19" extent="16-16"/>
 </signal>
 <signal name="N$9">
