File: layout/binaryclock.sch (EAGLE design)
At the start: 84 parts, among them IC1 LP2985, IC3 STM32F10XCXT6, Q1 BSS84, Q4 BC807-16SMD, X1 MINI-USB-SHIELD-UX60-MB-5ST

Commit message: split layout into three frames
Connections:
- removed net N$6: C3.1, IC3PORTC.PC15, XTAL.2
- removed net N$7: C2.2, IC3PORTC.PC14, XTAL.1
- new net OSC1: C2.2, XTAL.1
- new net OSC2: C3.1, XTAL.2
Other:
- note added: "Buttons"
- note added: "Buzzer"
- note added: "Crystal"
- note added: "Light Sensor"
- note added: "Power"
- note added: "Program Connector"
- note added: "Temperature Sensor"
- moved on the sheet: BATTERY, C10, C11, C12, C13, C14, C15, C16, C17, C18, C19, C2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
